File: Nebula - Master/Kicad/Watch/Nebula.kicad_sch (KiCad schematic)
At the start: 80 parts, among them J1 Female dock, J2 Display, M1 HMotor, Q1 s8050, Q2 CJ3139K, Q3 s8050, SW1 SW_Push, SW2 SW_Push, SW3 SW_Push, U1 XC3202B183MR-G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

Commit message: update
Connections:
- no-connect marks 6 -> 7
Changed lines of the file:
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@@
   (no_connect (at 245.11 199.39))
   (no_connect (at 245.11 194.31))
+  (no_connect (at 149.86 251.46))
   (no_connect (at 93.98 161.29))
   (no_connect (at 245.11 189.23))
