File: Nebula - Master/Kicad/Watch/Nebula.kicad_pcb (KiCad board)
At the start: 2 copper layers, 39.7 x 39.9 mm, 80 parts, among them J1 Female dock, J2 Display, M1 HMotor, Q1 s8050, Q2 CJ3139K, Q3 s8050, SW1 SW_Push, SW2 SW_Push, SW3 SW_Push, U1 XC3202B183MR-G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

Commit message: Added pcb images, schematic pdf and step
Parts:
- added G***: LOGO, somking:pumpkin2, B.Cu at (161.8, 94.8)
- added REF**: OSHW-Logo2_9.8x8mm_SilkScreen, Symbol:OSHW-Logo2_9.8x8mm_SilkScreen, B.Cu at (151.0, 74.8)
Other:
- board text added: "V2"

Commit message: update
Parts:
- moved J1 8.72 mm to (141.0, 90.7)
- moved F1 7.77 mm to (137.0, 90.8), turned to 0 degrees
- moved C15 6.26 mm to (142.5, 87.0), turned to 0 degrees
- moved 36 5.61 mm to (134.8, 90.5)
- moved PSU 4.27 mm to (137.2, 93.5)
- moved 39 2.36 mm to (138.0, 94.0)
- moved 38 1.97 mm to (134.8, 94.0)
- moved 37 1.36 mm to (138.0, 90.5)
- moved 41 1.35 mm to (138.0, 97.5)
- moved 40 0.96 mm to (134.8, 97.5)
- moved 35 0.36 mm to (138.2, 87.0)
- moved C11 0.30 mm to (142.5, 86.0)
Routing:
- net ESP_TX: track 12.7 -> 3.33 mm
- net ESP_RX: track 12.0 -> 3.56 mm
- net Net-(TP18-Pad1): track 3.87 -> 10.9 mm
- net Net-(TP21-Pad1): track 4.07 -> 6.85 mm
- net VCC_IN: track 13.3 -> 15.9 mm
- net PSU: track 10.2 -> 12.6 mm
- net Net-(TP20-Pad1): track 8.08 -> 10.2 mm
- net Net-(TP23-Pad1): track 6.55 -> 7.98 mm
- net Net-(TP22-Pad1): track 10.00 -> 10.9 mm
- net Net-(TP19-Pad1): track 8.20 -> 7.40 mm
- net GND: vias 11 -> 14
